Commit message: added right wheel to model

File: urdf/robot.urdf (robot description, URDF)
Before this commit: robot robot, 2 links, 1 joints
Links:
- added link link_right_wheel, mass 1; collision cylinder length=0.12 radius=0.08; collision cylinder length=0.12 radius=0.4
Joints:
- added joint joint_chassis_right_wheel: type continuous, parent link_chassis, child link_right_wheel, origin xyz=-0.5 -0.65 0 rpy=0 0 0, axis 0 1 0, limit effort=10000 velocity=1000

Commit message: added hubcaps to wheels to make spinning visible

File: urdf/robot.urdf (robot description, URDF)
Before this commit: robot robot, 3 links, 2 joints
Links:
- added link link_left_hubcap; visual box size=0.03 0.01 0.6
- added link link_right_hubcap; visual box size=0.03 0.01 0.6
Joints:
- added joint joint_left_wheel_left_hubcap: type fixed, parent link_left_wheel, child link_left_hubcap, origin xyz=0 0.24 0 rpy=0 0 0, axis 0 0 0
- added joint joint_right_wheel_right_hubcap: type fixed, parent link_right_wheel, child link_right_hubcap, origin xyz=0 -0.24 0 rpy=0 0 0, axis 0 0 0

Commit message: added castor wheel to model

File: urdf/robot.urdf (robot description, URDF)
Before this commit: robot robot, 5 links, 4 joints
Links:
- added link link_castor_wheel; visual sphere radius=0.125
Joints:
- added joint joint_chassis_castor_wheel: type fixed, parent link_chassis, child link_castor_wheel, origin xyz=0.875 0 -0.275 rpy=0 0 0, axis 0 0 0

Commit message: refactor to simplify robot model

File: urdf/robot.urdf (robot description, URDF)
Before this commit: robot robot, 6 links, 5 joints
Links:
- removed link link_left_hubcap
- removed link link_right_hubcap
- link link_castor_wheel: geometry collision sphere radius=0.125; visual sphere radius=0.125
- link link_left_wheel: geometry collision box size=0.03 0.01 0.6; collision cylinder length=0.12 radius=0.08
- link link_right_wheel: geometry collision box size=0.03 0.01 0.6; collision cylinder length=0.12 radius=0.08
Joints:
- removed joint joint_left_wheel_left_hubcap
- removed joint joint_right_wheel_right_hubcap

Commit message: replacing simple blocks with CAD mesh files

File: urdf/robot.urdf (robot description, URDF)
Before this commit: robot robot, 4 links, 3 joints
Links:
- link link_chassis: geometry collision box size=2 1.3 0.4; visual mesh filename=package://robot_description/meshes/chassis.stl
- link link_left_wheel: geometry collision box size=0.03 0.01 0.6; collision cylinder length=0.12 radius=0.4
- link link_right_wheel: geometry collision box size=0.03 0.01 0.6; collision cylinder length=0.12 radius=0.4

Commit message: set friction for wheels in gazebo

File: urdf/robot.urdf (robot description, URDF)
Before this commit: robot robot, 4 links, 3 joints
Links:
- removed link link_castor_wheel
- added link link_caster_wheel, mass 1; collision sphere radius=0.125; visual sphere radius=0.125
Joints:
- removed joint joint_chassis_castor_wheel
- added joint joint_chassis_caster_wheel: type fixed, parent link_chassis, child link_caster_wheel, origin xyz=0.875 0 -0.275 rpy=0 0 0
