Commit message: converted URDF file to XACRO and GAZEBO

File: urdf/robot.xacro (robot description, xacro)
@@ -1,114 +1,11 @@
 <?xml version="1.0" ?>
-<robot name="robot">
-    <!-- Gazebo - preserve caster -->
-    <gazebo reference="joint_chassis_caster_wheel">
-        <preserveFixedJoint>true</preserveFixedJoint>
-    </gazebo>
-    <!-- Gazebo - colors -->
-    <gazebo reference="link_chassis">
-        <material>Gazebo/Orange</material>
-    </gazebo>
-    <gazebo reference="link_caster_wheel">
-        <material>Gazebo/Black</material>
-        <mu1>0.0</mu1>
-        <mu2>0.0</mu2>
-    </gazebo>s
-    <gazebo reference="link_left_wheel">
-        <material>Gazebo/DarkGrey</material>
-        <mu1>0.2</mu1>
-        <mu2>0.2</mu2>
-    </gazebo>
-    <gazebo reference="link_right_wheel">
-        <material>Gazebo/DarkGrey</material>
-        <mu1>0.2</mu1>
-        <mu2>0.2</mu2>
-    </gazebo>
-    <!-- Gazebo - differential driver -->
-    <gazebo>
-        <plugin filename="libgazebo_ros_diff_drive.so" name="differential_drive_controller">
-            <alwaysOn>true</alwaysOn>
-            <updateRate>20</updateRate>
-            <leftJoint>joint_chassis_left_wheel</leftJoint>
-            <rightJoint>joint_chassis_right_wheel</rightJoint>
-            <wheelSeparation>1.66</wheelSeparation>
-            <wheelDiameter>0.8</wheelDiameter>
-            <torque>10</torque>
-            <commandTopic>cmd_vel</commandTopic>
-            <odometryTopic>odom</odometryTopic>
-            <odometryFrame>odom</odometryFrame>
-            <robotBaseFrame>link_chassis</robotBaseFrame>
-        </plugin>
-    </gazebo>
-    <!-- Gazebo tags - Laser scan -->
-    <gazebo reference="joint_laser_scan_chassis">
-        <preserveFixedJoint>true</preserveFixedJoint>
-    </gazebo>
-    <gazebo reference="link_laser_scan">
-        <material>Gazebo/DarkGrey</material>
-    </gazebo>
-    <gazebo reference="link_laser_scan">
-        <sensor type="ray" name="head_hokuyo_sensor">
-            <pose>0 0 0 0 0 0</pose>
-            <visualize>true</visualize>
-            <update_rate>20</update_rate>
-            <ray>
-                <scan>
-                    <horizontal>
-                        <samples>720</samples>
-                        <resolution>1</resolution>
-                        <min_angle>-1.570796</min_angle>
-                        <max_angle>1.570796</max_angle>
-                    </horizontal>
-                </scan>
-                <range>
-                    <min>0.20</min>
-                    <max>10.0</max>
-                    <resolution>0.01</resolution>
-                </range>
-                <noise>
-                    <type>gaussian</type>
-                    <mean>0.0</mean>
-                    <stddev>0.01</stddev>
-                </noise>
-            </ray>
-            <plugin name="gazebo_ros_head_hokuyo_controller" filename="libgazebo_ros_laser.so">
-                <topicName>/laser/scan</topicName>
-                <frameName>sensor_laser</frameName>
-            </plugin>
-        </sensor>
-    </gazebo>
-    <!-- URDF: Laser scan -->
-    <joint name="joint_laser_scan_chassis" type="fixed">
-        <origin rpy="0 0 0" xyz="0.8 0 0.3" />
-        <child link="link_laser_scan" />
-        <parent link="link_chassis" />
-        <joint_properties damping="1.0" friction="1.0" />
-    </joint>
-    <link name="link_laser_scan">
-        <inertial>
-            <origin xyz="0 0 0" rpy="0 0 0" />
-            <mass value="0.5" />
-            <inertia ixx="0.000252666666667" ixy="0" ixz="0" iyy="0.000252666666667" iyz="0" izz="0.0005"/>
-        </inertial>
-        <visual>
-            <origin xyz="0 0 0" rpy="0 0 0" />
-            <geometry>
-                <cylinder radius="0.15" length="0.20"/>
-            </geometry>
-            <material name="Red">
-                <color rgba="0.7 0.1 0.1 1" />
-            </material>
-        </visual>
-        <collision>
-            <origin xyz="0 0 0" rpy="0 0 0"/>
-            <geometry>
-                <cylinder radius="0.15" length="0.20"/>
-            </geometry>
-        </collision>
-    </link>
+<robot name="robot" xmlns:xacro="http://www.ros.org/wiki/xacro">
+    <xacro:include filename="$(find robot_description)/urdf/robot.gazebo" />
+    <!-- Parameters -->
+    <xacro:property name="chassis_mass" value="5" />
     <!-- Link - chassis -->
     <link name="link_chassis">
         <inertial>
-            <mass value="10" />
+            <mass value="${2 * chassis_mass}" />
             <origin xyz="0 0 0.3" rpy="0 0 0" />
             <inertia ixx="1.5417" ixy="0" ixz="0" iyy="3.467" iyz="0" izz="4.742" />
@@ -281,3 +178,33 @@
         </visual>
     </link>
+        <!-- Joint : Laser scan -->
+    <joint name="joint_laser_scan_chassis" type="fixed">
+        <origin rpy="0 0 0" xyz="0.8 0 0.3" />
+        <child link="link_laser_scan" />
+        <parent link="link_chassis" />
+        <joint_properties damping="1.0" friction="1.0" />
+    </joint>
+    <!-- Link : Laser scan -->
+    <link name="link_laser_scan">
+        <inertial>
+            <origin xyz="0 0 0" rpy="0 0 0" />
+            <mass value="0.5" />
+            <inertia ixx="0.000252666666667" ixy="0" ixz="0" iyy="0.000252666666667" iyz="0" izz="0.0005"/>
+        </inertial>
+        <visual>
+            <origin xyz="0 0 0" rpy="0 0 0" />
+            <geometry>
+                <cylinder radius="0.15" length="0.20"/>
+            </geometry>
+            <material name="Red">
+                <color rgba="0.7 0.1 0.1 1" />
+            </material>
+        </visual>
+        <collision>
+            <origin xyz="0 0 0" rpy="0 0 0"/>
+            <geometry>
+                <cylinder radius="0.15" length="0.20"/>
+            </geometry>
+        </collision>
+    </link>
 </robot>

Commit message: exerise completed: create pi property and replace angular values in XACRO with it

File: urdf/robot.xacro (robot description, xacro)
@@ -4,4 +4,5 @@
     <!-- Parameters -->
     <xacro:property name="chassis_mass" value="5" />
+    <xacro:property name="pi" value="3.1415" />
     <!-- Link - chassis -->
     <link name="link_chassis">
@@ -42,5 +43,5 @@
         </inertial>
         <collision>
-            <origin rpy="1.5707 0 0" xyz="0 0.18 0" />
+            <origin rpy="${pi / 2} 0 0" xyz="0 0.18 0" />
             <geometry>
                 <cylinder length="0.12" radius="0.4"/>
@@ -48,5 +49,5 @@
         </collision>
         <visual>
-            <origin rpy="1.5707 0 0" xyz="0 0.18 0" />
+            <origin rpy="${pi / 2} 0 0" xyz="0 0.18 0" />
             <geometry>
                 <mesh filename="package://robot_description/meshes/wheel.stl" />
@@ -57,26 +58,26 @@
         </visual>
         <collision>
-            <origin rpy="1.5707 0 0" xyz="0 0.06 0" />
-            <geometry>
-                <cylinder length="0.18" radius="0.08"/>
-            </geometry>
-        </collision>
-        <visual>
-            <origin rpy="1.5707 0 0" xyz="0 0.06 0" />
-            <geometry>
-                <cylinder length="0.18" radius="0.08"/>
-            </geometry>
-            <material name="White">
-                <color rgba="1 1 1 1" />
-            </material>
-        </visual>
-        <collision>
-            <origin rpy="0 0 0" xyz="0 0.18 0" />
-            <geometry>
-                <box size="0.03 0.01 0.6" />
-            </geometry>
-        </collision>
-        <visual>
-            <origin rpy="0 0 0" xyz="0 0.18 0" />
+            <origin rpy="${pi / 2} 0 0" xyz="0 0.06 0" />
+            <geometry>
+                <cylinder length="0.18" radius="0.08"/>
+            </geometry>
+        </collision>
+        <visual>
+            <origin rpy="${pi / 2} 0 0" xyz="0 0.06 0" />
+            <geometry>
+                <cylinder length="0.18" radius="0.08"/>
+            </geometry>
+            <material name="White">
+                <color rgba="1 1 1 1" />
+            </material>
+        </visual>
+        <collision>
+            <origin rpy="${pi / 2} 0 0" xyz="0 0.18 0" />
+            <geometry>
+                <box size="0.03 0.01 0.6" />
+            </geometry>
+        </collision>
+        <visual>
+            <origin rpy="${pi / 2} 0 0" xyz="0 0.18 0" />
             <geometry>
                 <box size="0.03 0.01 0.6" />
@@ -104,5 +105,5 @@
         </inertial>
         <collision>
-            <origin rpy="1.5707 0 0" xyz="0 -0.18 0" />
+            <origin rpy="${pi / 2} 0 0" xyz="0 -0.18 0" />
             <geometry>
                 <cylinder length="0.12" radius="0.4"/>
@@ -110,5 +111,5 @@
         </collision>
         <visual>
-            <origin rpy="1.5707 0 0" xyz="0 -0.18 0" />
+            <origin rpy="${pi / 2} 0 0" xyz="0 -0.18 0" />
             <geometry>
                 <mesh filename="package://robot_description/meshes/wheel.stl" />
@@ -119,26 +120,26 @@
         </visual>
         <collision>
-            <origin rpy="1.5707 0 0" xyz="0 -0.06 0" />
-            <geometry>
-                <cylinder length="0.18" radius="0.08"/>
-            </geometry>
-        </collision>
-        <visual>
-            <origin rpy="1.5707 0 0" xyz="0 -0.06 0" />
-            <geometry>
-                <cylinder length="0.18" radius="0.08"/>
-            </geometry>
-            <material name="White">
-                <color rgba="1 1 1 1" />
-            </material>
-        </visual>
-        <collision>
-            <origin rpy="0 0 0" xyz="0 -0.18 0" />
-            <geometry>
-                <box size="0.03 0.01 0.6" />
-            </geometry>
-        </collision>
-        <visual>
-            <origin rpy="0 0 0" xyz="0 -0.18 0" />
+            <origin rpy="${pi / 2} 0 0" xyz="0 -0.06 0" />
+            <geometry>
+                <cylinder length="0.18" radius="0.08"/>
+            </geometry>
+        </collision>
+        <visual>
+            <origin rpy="${pi / 2} 0 0" xyz="0 -0.06 0" />
+            <geometry>
+                <cylinder length="0.18" radius="0.08"/>
+            </geometry>
+            <material name="White">
+                <color rgba="1 1 1 1" />
+            </material>
+        </visual>
+        <collision>
+            <origin rpy="${pi / 2} 0 0" xyz="0 -0.18 0" />
+            <geometry>
+                <box size="0.03 0.01 0.6" />
+            </geometry>
+        </collision>
+        <visual>
+            <origin rpy="${pi / 2} 0 0" xyz="0 -0.18 0" />
             <geometry>
                 <box size="0.03 0.01 0.6" />

Commit message: added tail to robot and joint control scripts

File: urdf/robot.xacro (robot description, xacro)
@@ -209,3 +209,43 @@
         </collision>
     </link>
+    <!-- Robot tail -->
+    <joint name="joint_tail" type="continuous">
+        <origin rpy="0 0 0" xyz="-1 0 0" />
+        <child link="link_tail" />
+        <axis rpy="0 0 0" xyz="0 1 0" />
+        <parent link="link_chassis" />
+        <joint_properties damping="1.0" friction="1.0" />
+    </joint>
+    <link name="link_tail">
+        <inertial>
+            <origin xyz="0 0 0" rpy="0 0 0" />
+            <mass value="0.5" />
+            <inertia ixx="0.000252666666667" ixy="0" ixz="0" iyy="0.000252666666667" iyz="0" izz="0.0005"/>
+        </inertial>
+        <visual>
+            <origin xyz="-0.2 0 0" rpy="0 ${pi/2} 0" />
+            <geometry>
+                <cylinder radius="0.05" length="0.40"/>
+            </geometry>
+            <material name="Red">
+                <color rgba="0.7 0.1 0.1 1" />
+            </material>
+        </visual>
+        <collision>
+            <origin xyz="-0.2 0 0" rpy="0 ${pi/2} 0"/>
+            <geometry>
+                <cylinder radius="0.05" length="0.40"/>
+            </geometry>
+        </collision>
+    </link>
+    <transmission name="tran_tail">
+        <type>transmission_interface/SimpleTransmission</type>
+        <joint name="joint_tail">
+            <hardwareInterface>hardware_interface/EffortJointInterface</hardwareInterface>
+        </joint>
+        <actuator name="motor_joint_tail">
+            <hardwareInterface>hardware_interface/EffortJointInterface</hardwareInterface>
+            <mechanicalReduction>1</mechanicalReduction>
+        </actuator>
+    </transmission>
 </robot>
